File: Hardware/Arduino.kicad_pcb (KiCad board)
At the start: 2 copper layers, 40.6 x 76.2 mm, 17 parts, among them IC1 ATMEGA8-P, P1 CONN_5X2, P2 CONN_10, P3 CONN_10, P4 CONN_10, P5 CONN_10, SW1 SPST, X1 CRYSTAL

Commit message: added new files
Parts:
- added JP1: JUMPER, SIL-2, F.Cu at (105.4, 122.9)
- added LOGO: , logo:LOGO (2), F.Cu at (82.5, 67.0)
- added P6: CONN_7, SIL-7, F.Cu at (87.6, 120.4)
- SW1: footprint SW_PB_2pin_xl -> SW_PUSH_SMALL_2pin_xl
- moved D3 70.7 mm to (71.1, 60.7), turned to 180 degrees
- moved SW1 66.8 mm to (73.2, 122.4)
- moved R3 65.7 mm to (71.1, 56.9), turned to 0 degrees
- moved D2 65.0 mm to (71.1, 64.8)
- moved R1 41.6 mm to (103.4, 64.0)
- moved R2 41.4 mm to (78.2, 67.6), turned to 270 degrees
- moved D1 40.9 mm to (104.4, 58.9)
- moved IC1 40.7 mm to (87.6, 94.5)
- moved C1 40.4 mm to (96.8, 97.8)
- moved C2 40.2 mm to (97.0, 82.0)
- moved X1 40.1 mm to (97.3, 89.7)
- moved C3 39.9 mm to (79.2, 94.5)
- moved P2 39.1 mm to (69.8, 80.0)
- moved P3 39.1 mm to (69.8, 105.4)
- moved P4 39.1 mm to (105.4, 80.0)
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Connections:
- P4 pad 10: /9 -> /10
- P4 pad 6: /13 -> GND
- P4 pad 7: /12 -> /13
- P4 pad 8: /11 -> /12
- P4 pad 9: /10 -> /11
- P5 pad 1: /8 -> /9
- P5 pad 2: (no net) -> /8
Routing:
- net GND: track 159.4 -> 196.1 mm, vias 0 -> 4
- net /RESET: track 113.6 -> 148.3 mm
- net /VCC: track 101.9 -> 130.7 mm
- net /13: track 76.4 -> 55.4 mm
- net /TX: track 100.6 -> 117.5 mm
- net /AREF: track 71.2 -> 55.7 mm
- net N-0000023: track 0.00 -> 10.7 mm
- net /RX: track 93.9 -> 102.8 mm
- net /SDA: track 78.0 -> 84.9 mm
- net /SCL: track 83.4 -> 89.7 mm
- net /11: track 70.9 -> 65.4 mm, vias 3 -> 1
- net N-000006: track 12.5 -> 7.87 mm
- net /9: track 31.8 -> 35.7 mm
- net /8: track 23.9 -> 27.8 mm
- net /7: track 25.6 -> 28.5 mm
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- added copper zone on F.Cu, net /VCC
- added copper zone on B.Cu, net GND
Other:
- board size 40.6 x 76.2 mm -> 40 x 75 mm
- board text added: "A2"
- board text added: "DTR"
- board text added: "DTR JUMPER"
- board text removed: "A6"
- board text removed: "ARDUINO"

Commit message: added corrected files
Parts:
- removed LOGO: , logo:LOGO (2)
- added D4: LED, ee:LED-1206_NEW, F.Cu at (103.9, 65.5)
- added R4: 1k, Resistors_SMD:R_1206_HandSoldering, F.Cu at (71.6, 58.7)
- added R5: 1k, Resistors_SMD:R_1206_HandSoldering, F.Cu at (103.9, 62.7)
- D1, D2, D3: footprint SM1206 -> ee:LED-1206_NEW
- IC1: footprint DIP-28__300_ELL -> Sockets_DIP:DIP-28__300_ELL
- P1: footprint VASCH5x2 -> Connect:VASCH5x2
- R1, R2, R3: footprint SM1206 -> Resistors_SMD:R_1206_HandSoldering
- X1: footprint HC-49V -> Discret:HC-49V
- moved R3 5.11 mm to (71.6, 62.0)
- moved D3 4.83 mm to (71.1, 55.9)
- moved R1 4.35 mm to (103.9, 59.7)
- moved D1 2.59 mm to (103.9, 56.4), turned to 0 degrees
- moved R2 0.57 mm to (78.5, 68.1)
- moved D2 0.25 mm to (71.1, 65.0)
Connections:
- D2 pad 2: N-000006 -> Net-(D2-Pad2)
- D3 pad 2: N-000006 -> Net-(D3-Pad2)
- P1 pad 3: (no net) -> Net-(P1-Pad3)
- P2 pad 10: (no net) -> Net-(P2-Pad10)
- P2 pad 3: (no net) -> Net-(P2-Pad3)
- P2 pad 4: (no net) -> Net-(P2-Pad4)
- P2 pad 5: (no net) -> Net-(P2-Pad5)
- P2 pad 6: (no net) -> Net-(P2-Pad6)
- P2 pad 7: (no net) -> Net-(P2-Pad7)
- P2 pad 8: (no net) -> Net-(P2-Pad8)
- P2 pad 9: (no net) -> Net-(P2-Pad9)
- P3 pad 1: (no net) -> Net-(P3-Pad1)
- P3 pad 3: (no net) -> Net-(P3-Pad3)
- P3 pad 4: (no net) -> Net-(P3-Pad4)
- P6 pad 2: (no net) -> Net-(P6-Pad2)
- P6 pad 6: (no net) -> Net-(P6-Pad6)
- R3 pad 1: N-000006 -> Net-(D2-Pad2)
Routing:
- net /13: track 55.4 -> 71.0 mm, vias 1 -> 3
- net N-000006: track 7.87 -> 0.00 mm
- net /TX: track 117.5 -> 124.9 mm
- net GND: track 196.1 -> 202.0 mm, vias 4 -> 5
- net /VCC: track 130.7 -> 126.8 mm
- net Net-(D4-Pad2): track 0.00 -> 3.50 mm
- net Net-(D2-Pad2): track 0.00 -> 3.40 mm
- net Net-(D3-Pad2): track 0.00 -> 2.82 mm
Other:
- board text added: "(PWM*)"
- board text added: "*10"
- board text added: "*11"
- board text added: "*3"
- board text added: "*5"
- board text added: "*6"
- board text added: "*9"
- board text added: "PWR"
- board text removed: "10"
- board text removed: "11"
- board text removed: "3"
- board text removed: "5"
- board text removed: "6"
- board text removed: "9"

Commit message: added capacitor
Parts:
- removed JP1: JUMPER, SIL-2
- added C4: C, ee:SM1206, F.Cu at (103.9, 122.6)
- added LOGO: , logo:LOGO (2), B.Cu at (92.7, 66.7)
- C1, C2: footprint SM1206 -> ee:SM1206
- C3: footprint SM1206 -> ee:SM1206; moved to F.Cu
- moved C3 1.85 mm to (79.8, 96.3)
Routing:
- net GND: track 202.0 -> 206.5 mm
- net /SDA: track 84.9 -> 89.3 mm
- net /SCL: track 89.7 -> 94.0 mm
- net /RESET: track 148.4 -> 144.3 mm, vias 1 -> 2
Other:
- board text added: "Explore One for Arduino"
- board text removed: "DTR JUMPER"
